File: Converter_DC/Converter_DC.kicad_pcb (KiCad board)
At the start: 2 copper layers, 44.2 x 32.5 mm, 12 parts, among them J1 Screw_Terminal_01x02, J2 Screw_Terminal_01x02, U1 MC34063ECN

Commit message: add footprint
Parts:
- removed U1: MC34063ECN, DC-DC:DIP254P762X480-8
- added R1: 0, Resistor_THT:Resistor_L7.0mm_D2.5mm_d0.45mm, F.Cu at (153.1, 101.0)
- added RV1: 100k, Potentiometer_THT:TRIM_3296W-1-104, F.Cu at (161.5, 101.0)
- added U2: MC34063ECN, DC-DC:DIP254P762X480-8, F.Cu at (149.4, 95.4)
- L1: value 28uH -> 68uH
- R4: value 62k -> 150k
- moved R4 7.50 mm to (166.5, 101.0)
- moved J1 7.00 mm to (173.5, 103.5)
- moved R3 2.20 mm to (156.6, 101.0)
Connections:
- net /INPUT renamed /POWER_INPUT
- net /OUTPUT renamed /POWER_OUTPUT
- C1 pad 2: GND -> PGND
- C2 pad 2: GND -> SGND
- C3 pad 2: GND -> PGND
- J1 pad 1: GND -> PGND
- J2 pad 2: GND -> PGND
- R3 pad 1: GND -> SGND
Routing:
- net /POWER_OUTPUT: track 54.6 -> 71.8 mm
- net Net-(U2-CII): track 11.1 -> 20.1 mm
- net /POWER_INPUT: track 39.0 -> 46.9 mm
- added copper zone on B.Cu, net PGND
- added copper zone on F.Cu, net PGND
- added copper zone on F.Cu, net SGND
- removed copper zone on B.Cu, net GND
- removed copper zone on F.Cu, net GND
Other:
- board size 44.2 x 32.5 mm -> 52.4 x 32.5 mm
- board text removed: "R4"
