File: Converter_DC/Converter_DC.kicad_sch (KiCad schematic)
At the start: 12 parts, among them J1 Screw_Terminal_01x02, J2 Screw_Terminal_01x02, U1 MC34063ECN

Commit message: add footprint
Parts:
- removed U1: MC34063ECN, DC-DC:DIP254P762X480-8, symbol Converter_DCDC:MC34063ECN
- added R1: 0, Resistor_THT:Resistor_L7.0mm_D2.5mm_d0.45mm, symbol Device:R_US
- added R5: 25k, Resistor_THT:Resistor_L7.0mm_D2.5mm_d0.45mm, symbol Device:R_US
- added RV1: 100k, Potentiometer_THT:TRIM_3296W-1-104, symbol Device:R_Potentiometer
- added U2: MC34063ECN, DC-DC:DIP254P762X480-8, symbol DC-DC:MC34063ECN
- L1: value 28uH -> 68uH
- R4: value 62k -> 120k
Connections:
- net at R3.2, R4.2: now also R5.2, U2.5 (CII)
- net at D1.A, L1.2: now also U2.1 (SWC)
- net at C2.1: now also U2.3 (TC)
- net at L1.1, R2.1, RCS1.2: now also U2.7 (IPK)
- net at R2.2: now also U2.8 (DRC)
- net GND renamed PGND
- net PGND: now also R1.1, U2.2 (SWE), U2.4 (GND); no longer C2.2, R3.1
- net INPUT renamed POWER_INPUT
- net POWER_INPUT: now also U2.6 (VCC)
- net OUTPUT renamed POWER_OUTPUT
- net POWER_OUTPUT: now also RV1.2
- new net: R5.1, RV1.1
- new net SGND: C2.2, R1.2, R3.1
- no-connect marks 0 -> 1
Other:
- moved on the sheet: C1, C2, C3, D1, J1, J2, L1, R2, R3, RCS1
